Commit message: Oct 16th

File: ros_dd_simulation/ros_dd_description/urdf/ros_dd.urdf (robot description, URDF)
Before this commit: robot ros_dd_small, 7 links, 6 joints
Links:
- removed link caster_link_front
- removed link caster_link_rear
- added link front_caster_link, mass 0.1; collision sphere radius=0.03; visual sphere radius=0.03
- added link rear_caster_link, mass 0.1; collision sphere radius=0.03; visual sphere radius=0.03
- link laser_link: geometry collision box size=0.05 0.05 0.05; visual box size=0.05 0.05 0.05
- link left_wheel_link: mass 0.0625 -> 0.2
- link right_wheel_link: mass 0.0625 -> 0.2
Joints:
- removed joint caster_front_joint
- removed joint caster_rear_joint
- added joint front_caster_joint: type fixed, parent base_link, child front_caster_link, origin xyz=0.2 0 -0.045
- added joint rear_caster_joint: type fixed, parent base_link, child rear_caster_link, origin xyz=-0.2 0 -0.045
- joint laser_joint: origin xyz=0.3 0 0.15 rpy=0 0 0 -> xyz=0.25 0 0.16 rpy=0 0 0
- joint left_wheel_joint: origin xyz=0 0.175 -0.008 rpy=0 0 0 -> xyz=0 0.175 0 rpy=0 0 0
- joint right_wheel_joint: origin xyz=0 -0.175 -0.008 rpy=0 0 0 -> xyz=0 -0.175 0 rpy=0 0 0

File: ros_dd_simulation/ros_dd_description/urdf/ros_dd.xacro (robot description, xacro)
@@ -94,5 +94,5 @@
         <parent link="base_link"/>
         <child link="front_caster_link"/>
-        <origin xyz="${body_length/2 * 0.8} 0 -${body_height/2 - caster_radius}"/>
+        <origin xyz="${body_length/2 * 0.8} 0 -${wheel_radius - caster_radius}"/>
     </joint>
     <link name="rear_caster_link">
@@ -118,5 +118,5 @@
         <parent link="base_link"/>
         <child link="rear_caster_link"/>
-        <origin xyz="-${body_length/2 * 0.8} 0 -${body_height/2 - caster_radius}"/>
+        <origin xyz="-${body_length/2 * 0.8} 0 -${wheel_radius - caster_radius}"/>
     </joint>
     <link name="laser_link">
@@ -147,9 +147,7 @@
     </joint>
     <gazebo reference="base_link">
-        <material>Gazebo/Red</material>
         <self_collide>true</self_collide>
     </gazebo>
     <gazebo reference="left_wheel_link">
-        <material>Gazebo/Yellow</material>
         <mu1>1.0</mu1>
         <mu2>1.0</mu2>
@@ -158,5 +156,4 @@
     </gazebo>
     <gazebo reference="right_wheel_link">
-        <material>Gazebo/Yellow</material>
         <mu1>1.0</mu1>
         <mu2>1.0</mu2>
@@ -165,5 +162,4 @@
     </gazebo>
     <gazebo reference="front_caster_link">
-        <material>Gazebo/Grey</material>
         <mu1>0.0</mu1>
         <mu2>0.0</mu2>
@@ -172,5 +168,4 @@
     </gazebo>
     <gazebo reference="rear_caster_link">
-        <material>Gazebo/Grey</material>
         <mu1>0.0</mu1>
         <mu2>0.0</mu2>
@@ -178,55 +173,43 @@
         <minDepth>0.001</minDepth>
     </gazebo>
+    <!-- Gazebo Harmonic systems publish Gazebo Transport messages. -->
     <gazebo>
-        <plugin name="gazebo_ros_diff_drive" filename="libgazebo_ros_diff_drive.so">
-            <update_rate>50</update_rate>
+        <plugin filename="gz-sim-diff-drive-system" name="gz::sim::systems::DiffDrive">
             <left_joint>left_wheel_joint</left_joint>
             <right_joint>right_wheel_joint</right_joint>
-            <wheel_separation>${(body_width/2 + wheel_length/2) * 2}</wheel_separation>
-            <wheel_diameter>${wheel_radius*2}</wheel_diameter>
-            <max_wheel_torque>20</max_wheel_torque>
-            <max_wheel_acceleration>1.0</max_wheel_acceleration>
-            <ros>
-                <namespace></namespace>
-                <remapping>cmd_vel:=cmd_vel</remapping>
-                <remapping>odom:=odom</remapping>
-            </ros>
-            <odometry_frame>odom</odometry_frame>
-            <robot_base_frame>base_footprint</robot_base_frame>
-            <publish_odom>true</publish_odom>
-            <publish_odom_tf>true</publish_odom_tf>
-            <publish_wheel_tf>false</publish_wheel_tf>
+            <wheel_separation>${body_width + wheel_length}</wheel_separation>
+            <wheel_radius>${wheel_radius}</wheel_radius>
+            <topic>/cmd_vel</topic>
+            <odom_topic>/odom</odom_topic>
+            <tf_topic>/tf</tf_topic>
+            <frame_id>odom</frame_id>
+            <child_frame_id>base_footprint</child_frame_id>
+            <odom_publish_frequency>50</odom_publish_frequency>
+            <max_linear_acceleration>1.0</max_linear_acceleration>
+            <max_angular_acceleration>3.2</max_angular_acceleration>
         </plugin>
-    </gazebo>
-    <gazebo>
-        <plugin name="gazebo_ros_joint_state_publisher"
-                filename="libgazebo_ros_joint_state_publisher.so">
-            <ros>
-                <namespace></namespace>
-                <remapping>~/out:=joint_states</remapping>
-            </ros>
-            <update_rate>50</update_rate>
+        <plugin filename="gz-sim-joint-state-publisher-system"
+                name="gz::sim::systems::JointStatePublisher">
+            <topic>/joint_states</topic>
             <joint_name>left_wheel_joint</joint_name>
             <joint_name>right_wheel_joint</joint_name>
         </plugin>
     </gazebo>
-    <gazebo>
-        <plugin name="imu_plugin" filename="libgazebo_ros_imu.so">
-            <alwaysOn>true</alwaysOn>
-            <updateRate>100.0</updateRate>
-            <bodyName>base_link</bodyName>
-            <topicName>imu/data</topicName>
-            <gaussianNoise>0.005</gaussianNoise>
-            <xyzOffset>0 0 0</xyzOffset>
-            <rpyOffset>0 0 0</rpyOffset>
-        </plugin>
+    <gazebo reference="base_link">
+        <sensor name="imu_sensor" type="imu">
+            <always_on>true</always_on>
+            <update_rate>100</update_rate>
+            <topic>/imu/data</topic>
+            <gz_frame_id>base_link</gz_frame_id>
+            <imu/>
+        </sensor>
     </gazebo>
     <gazebo reference="laser_link">
-        <sensor type="ray" name="laser_sensor">
+        <sensor type="gpu_lidar" name="laser_sensor">
             <pose>0 0 0 0 0 0</pose>
             <visualize>true</visualize>
             <update_rate>10</update_rate>
             <always_on>1</always_on>
-            <ray>
+            <lidar>
                 <scan>
                     <horizontal>
@@ -247,13 +230,7 @@
                     <stddev>0.01</stddev>
                 </noise>
-            </ray>
-            <plugin name="gazebo_ros_laser_controller" filename="libgazebo_ros_ray_sensor.so">
-                <ros>
-                    <namespace></namespace>
-                    <remapping>~/out:=scan</remapping>
-                </ros>
-                <output_type>sensor_msgs/LaserScan</output_type>
-                <frame_name>laser_link</frame_name>
-            </plugin>
+            </lidar>
+            <topic>/scan</topic>
+            <gz_frame_id>laser_link</gz_frame_id>
         </sensor>
     </gazebo>
